File: eagle-6502/base/base.brd (EAGLE design)
At the start: 160 x 99.1 mm, 146 parts, among them M1 ARDUINO_MEGA_PINS, M2 LCD-16X2, U1 W65C02S6TP, U2 28C256, U3 62256, U4 W65C22S6TP, U5 74HC00N, U6 74138N, U7 74HC00N, X13 TACT_SWITCH, X14 TACT_SWITCH, X15 TACT_SWITCH, X16 TACT_SWITCH, X6 TACT_SWITCH, X7 TACT_SWITCH

Commit message: Terminal Feature Complete
Connections:
- new net EEPROM_!OE: M1.38, U2.22
- net GND: no longer U2.22
Changed lines of the file:
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@@
 <contactref element="C3" pad="2"/>
 <contactref element="U3" pad="14"/>
-<contactref element="U2" pad="22"/>
 <contactref element="M2" pad="1"/>
 <contactref element="M2" pad="16"/>
@@
 <via x="149.86" y="46.99" extent="1-16" drill="0.5"/>
 <via x="154.94" y="54.61" extent="1-16" drill="0.5"/>
+<wire x1="116.84" y1="78.74" x2="124.46" y2="96.52" width="0" layer="19" extent="1-1"/>
+<wire x1="104.14" y1="78.74" x2="116.84" y2="78.74" width="0" layer="19" extent="1-1"/>
+<wire x1="93.98" y1="78.74" x2="104.14" y2="78.74" width="0" layer="19" extent="1-1"/>
+<wire x1="86.36" y1="96.52" x2="93.98" y2="78.74" width="0" layer="19" extent="1-1"/>
+<wire x1="74.93" y1="96.2" x2="86.36" y2="96.52" width="0" layer="19" extent="1-1"/>
+<wire x1="74.93" y1="97.79" x2="74.93" y2="96.2" width="0" layer="19" extent="1-1"/>
+<wire x1="67.056" y1="96.52" x2="74.93" y2="96.2" width="0" layer="19" extent="1-1"/>
+<wire x1="66.36" y1="93.98" x2="67.056" y2="96.52" width="0" layer="19" extent="1-1"/>
+<wire x1="57.15" y1="93.98" x2="66.36" y2="93.98" width="0" layer="19" extent="1-1"/>
+<wire x1="56.2" y1="87.63" x2="57.15" y2="93.98" width="0" layer="19" extent="1-1"/>
+<wire x1="45.72" y1="76.2" x2="56.2" y2="87.63" width="0" layer="19" extent="1-1"/>
+<wire x1="38.1" y1="78.74" x2="45.72" y2="76.2" width="0" layer="19" extent="1-1"/>
+<wire x1="31.75" y1="78.74" x2="38.1" y2="78.74" width="0" layer="19" extent="1-1"/>
+<wire x1="25.4" y1="76.2" x2="31.75" y2="78.74" width="0" layer="19" extent="1-1"/>
+<wire x1="22.86" y1="78.74" x2="25.4" y2="76.2" width="0" layer="19" extent="1-1"/>
+<wire x1="13.97" y1="78.74" x2="22.86" y2="78.74" width="0" layer="19" extent="1-1"/>
+<wire x1="28.26" y1="87.63" x2="31.75" y2="78.74" width="0" layer="19" extent="1-1"/>
+<wire x1="20.32" y1="66.04" x2="25.4" y2="76.2" width="0" layer="19" extent="1-1"/>
+<wire x1="20.32" y1="60.96" x2="20.32" y2="66.04" width="0" layer="19" extent="1-1"/>
+<wire x1="20.32" y1="50.8" x2="20.32" y2="60.96" width="0" layer="19" extent="1-1"/>
+<wire x1="8.89" y1="59.055" x2="20.32" y2="60.96" width="0" layer="19" extent="1-1"/>
+<wire x1="3.81" y1="58.42" x2="8.89" y2="59.055" width="0" layer="19" extent="1-1"/>
+<wire x1="7.94" y1="50.8" x2="8.89" y2="59.055" width="0" layer="19" extent="1-1"/>
+<wire x1="3.81" y1="33.02" x2="3.81" y2="44.45" width="0" layer="19" extent="1-1"/>
+<wire x1="7.62" y1="88.58" x2="13.97" y2="78.74" width="0" layer="19" extent="1-1"/>
+<wire x1="5.08" y1="93.98" x2="7.62" y2="88.58" width="0" layer="19" extent="1-1"/>
+<wire x1="19.05" y1="96.012" x2="28.26" y2="87.63" width="0" layer="19" extent="1-1"/>
+<wire x1="69.85" y1="78.74" x2="66.36" y2="93.98" width="0" layer="19" extent="1-1"/>
+<wire x1="72.39" y1="78.74" x2="69.85" y2="78.74" width="0" layer="19" extent="1-1"/>
+<wire x1="73.66" y1="76.2" x2="72.39" y2="78.74" width="0" layer="19" extent="1-1"/>
+<wire x1="38.1" y1="52.07" x2="20.32" y2="50.8" width="0" layer="19" extent="1-1"/>
+<wire x1="38.1" y1="48.26" x2="38.1" y2="52.07" width="0" layer="19" extent="1-1"/>
+<wire x1="71.12" y1="53.34" x2="73.66" y2="76.2" width="0" layer="19" extent="1-1"/>
+<wire x1="93.98" y1="53.34" x2="71.12" y2="53.34" width="0" layer="19" extent="1-1"/>
+<wire x1="106.68" y1="43.18" x2="93.98" y2="53.34" width="0" layer="19" extent="1-1"/>
+<wire x1="106.68" y1="38.1" x2="106.68" y2="43.18" width="0" layer="19" extent="1-1"/>
+<wire x1="113.03" y1="28.89" x2="106.68" y2="38.1" width="0" layer="19" extent="1-1"/>
+<wire x1="113.7412" y1="19.3294" x2="113.03" y2="28.89" width="0" layer="19" extent="1-1"/>
+<wire x1="107.2388" y1="19.3294" x2="113.7412" y2="19.3294" width="0" layer="19" extent="1-1"/>
+<wire x1="121.2088" y1="19.3294" x2="113.7412" y2="19.3294" width="0" layer="19" extent="1-1"/>
+<wire x1="127.7112" y1="19.3294" x2="121.2088" y2="19.3294" width="0" layer="19" extent="1-1"/>
+<wire x1="135.1788" y1="19.3294" x2="127.7112" y2="19.3294" width="0" layer="19" extent="1-1"/>
+<wire x1="141.6812" y1="19.3294" x2="135.1788" y2="19.3294" width="0" layer="19" extent="1-1"/>
+<wire x1="149.1488" y1="19.3294" x2="141.6812" y2="19.3294" width="0" layer="19" extent="1-1"/>
+<wire x1="155.6512" y1="19.3294" x2="149.1488" y2="19.3294" width="0" layer="19" extent="1-1"/>
+<wire x1="154.94" y1="28.89" x2="155.6512" y2="19.3294" width="0" layer="19" extent="1-1"/>
+<wire x1="156.21" y1="38.42" x2="156.21" y2="29.21" width="0" layer="19" extent="1-1"/>
+<wire x1="149.86" y1="38.1" x2="156.21" y2="38.42" width="0" layer="19" extent="1-1"/>
+<wire x1="149.86" y1="46.99" x2="149.86" y2="38.1" width="0" layer="19" extent="1-1"/>
+<wire x1="154.94" y1="54.61" x2="149.86" y2="46.99" width="0" layer="19" extent="1-1"/>
+<wire x1="140.97" y1="28.89" x2="141.6812" y2="19.3294" width="0" layer="19" extent="1-1"/>
+<wire x1="127" y1="28.89" x2="127.7112" y2="19.3294" width="0" layer="19" extent="1-1"/>
+<wire x1="121.285" y1="9.525" x2="121.2088" y2="19.3294" width="0" layer="19" extent="1-1"/>
+<wire x1="123.19" y1="5.4" x2="121.285" y2="9.525" width="0" layer="19" extent="1-1"/>
+<wire x1="121.92" y1="2.54" x2="123.19" y2="5.4" width="0" layer="19" extent="1-1"/>
+<wire x1="118.11" y1="5.4" x2="121.92" y2="2.54" width="0" layer="19" extent="1-1"/>
+<wire x1="115.57" y1="5.4" x2="118.11" y2="5.4" width="0" layer="19" extent="1-1"/>
+<wire x1="113.03" y1="5.4" x2="115.57" y2="5.4" width="0" layer="19" extent="1-1"/>
+<wire x1="110.49" y1="5.4" x2="113.03" y2="5.4" width="0" layer="19" extent="1-1"/>
+<wire x1="107.95" y1="5.4" x2="110.49" y2="5.4" width="0" layer="19" extent="1-1"/>
+<wire x1="105.41" y1="5.4" x2="107.95" y2="5.4" width="0" layer="19" extent="1-1"/>
+<wire x1="102.87" y1="5.4" x2="105.41" y2="5.4" width="0" layer="19" extent="1-1"/>
+<wire x1="100.33" y1="5.4" x2="102.87" y2="5.4" width="0" layer="19" extent="1-1"/>
+<wire x1="99.06" y1="2.54" x2="100.33" y2="5.4" width="0" layer="19" extent="1-1"/>
+<wire x1="98.425" y1="9.525" x2="100.33" y2="5.4" width="0" layer="19" extent="1-1"/>
+<wire x1="95.25" y1="5.4" x2="99.06" y2="2.54" width="0" layer="19" extent="1-1"/>
+<wire x1="92.71" y1="5.4" x2="95.25" y2="5.4" width="0" layer="19" extent="1-1"/>
+<wire x1="90.17" y1="5.4" x2="92.71" y2="5.4" width="0" layer="19" extent="1-1"/>
+<wire x1="87.63" y1="5.4" x2="90.17" y2="5.4" width="0" layer="19" extent="1-1"/>
+<wire x1="85.09" y1="5.4" x2="87.63" y2="5.4" width="0" layer="19" extent="1-1"/>
+<wire x1="82.55" y1="5.4" x2="85.09" y2="5.4" width="0" layer="19" extent="1-1"/>
+<wire x1="80.01" y1="5.4" x2="82.55" y2="5.4" width="0" layer="19" extent="1-1"/>
+<wire x1="77.47" y1="5.4" x2="80.01" y2="5.4" width="0" layer="19" extent="1-1"/>
+<wire x1="74.93" y1="5.4" x2="77.47" y2="5.4" width="0" layer="19" extent="1-1"/>
+<wire x1="72.39" y1="5.4" x2="74.93" y2="5.4" width="0" layer="19" extent="1-1"/>
+<wire x1="69.85" y1="5.4" x2="72.39" y2="5.4" width="0" layer="19" extent="1-1"/>
+<wire x1="67.31" y1="5.4" x2="69.85" y2="5.4" width="0" layer="19" extent="1-1"/>
+<wire x1="64.77" y1="5.4" x2="67.31" y2="5.4" width="0" layer="19" extent="1-1"/>
+<wire x1="62.23" y1="5.4" x2="64.77" y2="5.4" width="0" layer="19" extent="1-1"/>
+<wire x1="59.69" y1="5.4" x2="62.23" y2="5.4" width="0" layer="19" extent="1-1"/>
+<wire x1="57.15" y1="5.4" x2="59.69" y2="5.4" width="0" layer="19" extent="1-1"/>
+<wire x1="54.61" y1="2.54" x2="57.15" y2="5.4" width="0" layer="19" extent="1-1"/>
+<wire x1="130.81" y1="5.4" x2="123.19" y2="5.4" width="0" layer="19" extent="1-1"/>
+<wire x1="135.1788" y1="7.8994" x2="130.81" y2="5.4" width="0" layer="19" extent="1-1"/>
+<wire x1="141.6812" y1="7.8994" x2="135.1788" y2="7.8994" width="0" layer="19" extent="1-1"/>
+<wire x1="142.24" y1="2.54" x2="141.6812" y2="7.8994" width="0" layer="19" extent="1-1"/>
+<wire x1="139.7" y1="2.54" x2="142.24" y2="2.54" width="0" layer="19" extent="1-1"/>
+<wire x1="146.05" y1="4.13" x2="142.24" y2="2.54" width="0" layer="19" extent="1-1"/>
+<wire x1="149.1488" y1="7.8994" x2="146.05" y2="4.13" width="0" layer="19" extent="1-1"/>
+<wire x1="155.6512" y1="7.8994" x2="149.1488" y2="7.8994" width="0" layer="19" extent="1-1"/>
+<wire x1="95.25" y1="16.51" x2="98.425" y2="9.525" width="0" layer="19" extent="1-1"/>
+<wire x1="52.07" y1="11.43" x2="57.15" y2="5.4" width="0" layer="19" extent="1-1"/>
+<wire x1="49.53" y1="11.43" x2="52.07" y2="11.43" width="0" layer="19" extent="1-1"/>
+<wire x1="53.66" y1="16.51" x2="52.07" y2="11.43" width="0" layer="19" extent="1-1"/>
+<wire x1="86.04" y1="16.51" x2="95.25" y2="16.51" width="0" layer="19" extent="1-1"/>
+<wire x1="124.46" y1="46.99" x2="106.68" y2="43.18" width="0" layer="19" extent="1-1"/>
+<wire x1="30.48" y1="20.32" x2="49.53" y2="11.43" width="0" layer="19" extent="1-1"/>
+<wire x1="27.94" y1="12.7" x2="30.48" y2="20.32" width="0" layer="19" extent="1-1"/>
+<wire x1="15.24" y1="9.84" x2="27.94" y2="12.7" width="0" layer="19" extent="1-1"/>
+<wire x1="7.62" y1="9.84" x2="15.24" y2="9.84" width="0" layer="19" extent="1-1"/>
+<wire x1="7.62" y1="5.08" x2="7.62" y2="9.84" width="0" layer="19" extent="1-1"/>
+<wire x1="7.62" y1="2.54" x2="7.62" y2="5.08" width="0" layer="19" extent="1-1"/>
+<wire x1="142.24" y1="78.74" x2="124.46" y2="96.52" width="0" layer="19" extent="1-1"/>
 </signal>
 <signal name="RDY">
@@
 <wire x1="66.675" y1="91.44" x2="90.17" y2="91.44" width="0.4" layer="1"/>
 </signal>
+<signal name="EEPROM_!OE">
+<contactref element="U2" pad="22"/>
+<contactref element="M1" pad="38"/>
+<wire x1="27.94" y1="5.08" x2="55.88" y2="35.56" width="0" layer="19" extent="1-1"/>
+</signal>
 </signals>
