File: eagle-6502/base/base.sch (EAGLE design)
At the start: 146 parts, among them M1 ARDUINO_MEGA_PINS, M2 LCD-16X2, U1 W65C02S6TP, U2 28C256, U3 62256, U4 W65C22S6TP, U5 74HC00N, U6 74138N, U7 74HC00N, X13 TACT_SWITCH, X14 TACT_SWITCH, X15 TACT_SWITCH, X16 TACT_SWITCH, X6 TACT_SWITCH, X7 TACT_SWITCH

Commit message: Terminal Feature Complete
Connections:
- new net EEPROM_!OE: M1.PD7, U2.!OE
- net GND: no longer U2.!OE
Changed lines of the file:
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@@
 <part name="GND7" library="supply1" library_urn="urn:adsk.eagle:library:371" deviceset="GND" device=""/>
 <part name="U3" library="6502_lib" deviceset="62256" device="" package3d_urn="urn:adsk.eagle:package:20790/1"/>
-<part name="GND8" library="supply1" library_urn="urn:adsk.eagle:library:371" deviceset="GND" device=""/>
 <part name="M2" library="6502_lib" deviceset="LCD-16X2" device=""/>
 <part name="P+6" library="supply1" library_urn="urn:adsk.eagle:library:371" deviceset="+5V" device=""/>
@@
 <attribute name="VALUE" x="139.7" y="-7.62" size="1.778" layer="96"/>
 </instance>
-<instance part="GND8" gate="1" x="35.56" y="-27.94" smashed="yes">
-<attribute name="VALUE" x="33.02" y="-30.48" size="1.778" layer="96"/>
-</instance>
 <instance part="M2" gate="G$1" x="165.1" y="-114.3" smashed="yes">
 <attribute name="NAME" x="157.48" y="-93.98" size="1.778" layer="95"/>
@@
 </segment>
 <segment>
-<pinref part="U2" gate="G$1" pin="!OE"/>
-<wire x1="53.34" y1="-20.32" x2="35.56" y2="-20.32" width="0.1524" layer="91"/>
-<wire x1="35.56" y1="-20.32" x2="35.56" y2="-25.4" width="0.1524" layer="91"/>
-<pinref part="GND8" gate="1" pin="GND"/>
-</segment>
-<segment>
 <pinref part="GND9" gate="1" pin="GND"/>
 <wire x1="149.86" y1="-132.08" x2="149.86" y2="-129.54" width="0.1524" layer="91"/>
@@
 </segment>
 </net>
+<net name="EEPROM_!OE" class="0">
+<segment>
+<pinref part="U2" gate="G$1" pin="!OE"/>
+<wire x1="53.34" y1="-20.32" x2="50.8" y2="-20.32" width="0.1524" layer="91"/>
+<label x="50.8" y="-20.32" size="1.27" layer="95" rot="R180" xref="yes"/>
+</segment>
+<segment>
+<pinref part="M1" gate="G$1" pin="PD7"/>
+<wire x1="17.78" y1="66.04" x2="15.24" y2="66.04" width="0.1524" layer="91"/>
+<label x="15.24" y="66.04" size="1.27" layer="95" rot="R180" xref="yes"/>
+</segment>
+</net>

Commit message: Updated Schematic, Added PDF
Other:
- note added: "6502 Peripherals: EEPROM, RAM, PIA, LCD"
- note added: "Address Decoding"
- note added: "Arduino Mega Pinout and 6502 Processor"
- note added: "Status LEDs and Connectors"
